Commit message: inertia added

File: robotiq_hande_description/urdf/robotiq_hande.urdf.xacro (robot description, xacro)
@@ -10,6 +10,5 @@
       <inertial>
         <origin xyz="0 0 0.04607" rpy="${pi/2} 0 ${pi/2}" />
-        <mass value="0.86387" />
-        <inertia ixx="1017560E-9" ixy="0" ixz="2235E-9" iyy="1028041E-9" iyz="0" izz="489810E-9" />
+s
       </inertial>
       <visual>
